Commit message: solve escape room fixed + room2 added, green goal mark for robot added, benchmark room fix coming next

File: robowflex_dart/include/io/envs/fetch/urdf/fetch3.urdf (robot description, URDF)
Before this commit: robot fetch, 28 links, 27 joints
Links:
- added link rotate_z_axis
Joints:
- added joint rotate_z_joint: type revolute, parent rotate_z_axis, child base_link, origin xyz=0 0 0 rpy=0 0 0, axis 0 0 1, limit lower=-3.14 upper=3.14 effort=10 velocity=20
- joint move_x_axis_joint: child base_link -> move_y_axis; limit lower=-1.5 upper=3.0 effort=10000 velocity=20 -> lower=-5.0 upper=5.0 effort=10 velocity=20
- joint move_y_axis_joint: child move_y_axis -> rotate_z_axis; limit lower=-3.0 upper=3.0 effort=10000 velocity=20 -> lower=-5.0 upper=5.0 effort=10 velocity=20; parent move_x_axis -> move_y_axis

File: robowflex_dart/include/io/envs/room/urdf/room.urdf (robot description, URDF)
Before this commit: robot escape_scene, 12 links, 11 joints
Links:
- removed link cube1
- removed link cube2
- removed link door_lock
- removed link front_door
- added link goal; visual cylinder length=0.001 radius=0.25
- added link link_0_joint_0; collision box size=0.5 0.5 0.75; visual box size=0.5 0.5 0.75
- added link link_1_joint_0; collision box size=0.5 0.5 0.75; visual box size=0.5 0.5 0.75
- added link link_2_joint_0; collision box size=0.1 0.7 1.1; visual box size=0.1 0.7 1.1
- added link link_3_joint_0; collision box size=0.03 0.45 0.146; visual box size=0.03 0.45 0.146
- link desk: geometry collision mesh filename=file:///home/serboba/rb_ws/src/robowflex/robowflex_dart/inc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 scale=0.01 0.01 0.020; visual mesh filename=file:///home/serboba/rb_ws/src/robowflex/robowflex_dart/inc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 scale=0.01 0.01 0.020
- link room: geometry collision mesh filename=file:///home/serboba/rb_ws/src/robowflex/robowflex_dart/inc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 scale=0.4 0.4 0.3; visual mesh filename=file:///home/serboba/rb_ws/src/robowflex/robowflex_dart/inc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 scale=0.4 0.4 0.3
- link shelf: geometry collision mesh filename=file:///home/serboba/rb_ws/src/robowflex/robowflex_dart/inc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 scale=0.042 0.05 0.04; visual mesh filename=file:///home/serboba/rb_ws/src/robowflex/robowflex_dart/inc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 scale=0.042 0.05 0.04
- link sofa: geometry collision mesh filename=file:///home/serboba/rb_ws/src/robowflex/robowflex_dart/inc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 scale=0.7 0.7 1; visual mesh filename=file:///home/serboba/rb_ws/src/robowflex/robowflex_dart/inc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 scale=0.7 0.7 1
Joints:
- removed joint cube1_joint
- removed joint cube1_joint2
- removed joint cube2_joint
- removed joint cube2_joint2
- removed joint door_lock_joint
- removed joint front_door_joint
- added joint goal: type fixed, parent base_link, child goal, origin xyz=2.0 0 0 rpy=0 0 0
- added joint link_0_joint_0: type prismatic, parent base_link, child cube1_y_axis, origin xyz=0.95 0.1 0.375 rpy=0 0 0, axis 0 1 0, limit lower=-1.10 upper=0.96 effort=0.05 velocity=1.57
- added joint link_0_joint_1: type prismatic, parent cube1_y_axis, child link_0_joint_0, origin xyz=0 0 0 rpy=0 0 0, axis 1 0 0, limit lower=-1.5 upper=0.05 effort=0.05 velocity=1.57
- added joint link_1_joint_0: type prismatic, parent base_link, child cube2_y_axis, origin xyz=0.95 -0.9 0.375 rpy=0 0 0, axis 0 1 0, limit lower=-0.1 upper=1.90 effort=0.05 velocity=1.57
- added joint link_1_joint_1: type prismatic, parent cube2_y_axis, child link_1_joint_0, origin xyz=0 0 0 rpy=0 0 0, axis 1 0 0, limit lower=-1.5 upper=0.05 effort=0.05 velocity=1.57
- added joint link_2_joint_0: type revolute, parent base_link, child link_2_joint_0, origin xyz=1.30 -0.4 0.55 rpy=0 0 0, axis 0 0 1, limit lower=0 upper=1.57 effort=0.05 velocity=1.57
- added joint link_3_joint_0: type revolute, parent base_link, child link_3_joint_0, origin xyz=1.22 0.45 0.90 rpy=0 0 0, axis 1 0 0, limit lower=0 upper=1.57 effort=0.05 velocity=1.57
