Commit message: solve escape room script fixed, benchmark room fixed, fetch x-y bounds for escape room scenarios adjusted, room2 added to demonstrate limitations

File: robowflex_dart/include/io/envs/fetch/urdf/fetch2.urdf (robot description, URDF)
Before this commit: robot fetch, 28 links, 27 joints
Joints:
- joint move_x_axis_joint: limit lower=-1.1 upper=2.1 effort=10 velocity=20 -> lower=-1.1 upper=2.25 effort=10 velocity=20
- joint move_y_axis_joint: limit lower=-1.0 upper=1.1 effort=10 velocity=20 -> lower=-1.1 upper=1.1 effort=10 velocity=20

File: robowflex_dart/include/io/envs/room0/urdf/room0.urdf (robot description, URDF)
Before this commit: robot room, 13 links, 12 joints
Links:
- link desk: geometry collision mesh filename=file:///home/serboba/Desktop/blenderFLEX/desk2.dae scale=0.01 0.01 0.020; visual mesh filename=file:///home/serboba/Desktop/blenderFLEX/desk2.dae scale=0.01 0.01 0.020
- link room: geometry collision mesh filename=file:///home/serboba/Desktop/blenderFLEX/room.dae scale=0.4 0.4 0.3; visual mesh filename=file:///home/serboba/Desktop/blenderFLEX/room.dae scale=0.4 0.4 0.3
- link shelf: geometry collision mesh filename=file:///home/serboba/Desktop/blenderFLEX/shelf.dae scale=0.042 0.05 0.04; visual mesh filename=file:///home/serboba/Desktop/blenderFLEX/shelf.dae scale=0.042 0.05 0.04
- link sofa: geometry collision mesh filename=file:///home/serboba/Desktop/blenderFLEX/sofa.dae scale=0.7 0.7 1; visual mesh filename=file:///home/serboba/Desktop/blenderFLEX/sofa.dae scale=0.7 0.7 1
Joints:
- joint goal: origin xyz=2.0 0 0.0 rpy=0 0 0 -> xyz=2.0 0.0 0.0 rpy=0 0 0

File: robowflex_dart/include/io/envs/room1/urdf/room1.urdf (robot description, URDF)
Before this commit: robot room, 13 links, 12 joints
Links:
- link desk: geometry collision mesh filename=file:///home/serboba/Desktop/blenderFLEX/desk2.dae scale=0.01 0.01 0.020; visual mesh filename=file:///home/serboba/Desktop/blenderFLEX/desk2.dae scale=0.01 0.01 0.020
- link link_0_joint_0: geometry collision box size=0.4 0.65 0.75; visual box size=0.4 0.65 0.75
- link link_1_joint_0: geometry collision box size=0.4 0.5 0.75; visual box size=0.4 0.5 0.75
- link room: geometry collision mesh filename=file:///home/serboba/Desktop/blenderFLEX/room.dae scale=0.4 0.4 0.3; visual mesh filename=file:///home/serboba/Desktop/blenderFLEX/room.dae scale=0.4 0.4 0.3
- link shelf: geometry collision mesh filename=file:///home/serboba/Desktop/blenderFLEX/shelf.dae scale=0.042 0.05 0.04; visual mesh filename=file:///home/serboba/Desktop/blenderFLEX/shelf.dae scale=0.042 0.05 0.04
- link sofa: geometry collision mesh filename=file:///home/serboba/Desktop/blenderFLEX/sofa.dae scale=0.9 0.7 1; visual mesh filename=file:///home/serboba/Desktop/blenderFLEX/sofa.dae scale=0.9 0.7 1
Joints:
- joint desk_joint: origin xyz=0.30 0.6 0.0 rpy=0 0 1.57 -> xyz=0.25 0.6 0.0 rpy=0 0 1.57
- joint goal: origin xyz=2.0 0 0.0 rpy=0 0 0 -> xyz=2.0 0.0 0.0 rpy=0 0 0
- joint link_0_joint_0: limit lower=-1.10 upper=0.96 effort=0.05 velocity=1.57 -> lower=-0.60 upper=1.10 effort=0.05 velocity=1.57; origin xyz=0.95 0.1 0.375 rpy=0 0 0 -> xyz=-0.5 -0.1 0.375 rpy=0 0 0
- joint link_0_joint_1: limit lower=-1.5 upper=0.05 effort=0.05 velocity=1.57 -> lower=-1.0 upper=1.65 effort=0.05 velocity=1.57
- joint link_1_joint_0: limit lower=-0.1 upper=1.90 effort=0.05 velocity=1.57 -> lower=-1.15 upper=0.95 effort=0.05 velocity=1.57; origin xyz=0.95 -0.9 0.375 rpy=0 0 0 -> xyz=0.95 0.1 0.375 rpy=0 0 0
- joint link_1_joint_1: limit lower=-1.5 upper=0.05 effort=0.05 velocity=1.57 -> lower=-2.10 upper=0.15 effort=0.05 velocity=1.57
- joint sofa_joint: origin xyz=-0.90 -0.2 0.0 rpy=0 0 1.57 -> xyz=-0.3 -1.0 0.0 rpy=0 0 -3.14
