Commit message: LA-RRT fixed bugs, optimized better solution (+trySkipFragment), memleaks fixed, manipulation bug fixes, fetch urdf joints and bounds bug fixes

File: robowflex_dart/include/io/envs/fetch/urdf/fetch4.urdf (robot description, URDF)
Before this commit: robot fetch, 29 links, 28 joints
Links:
- link base_link: geometry collision mesh filename=file:///home/serboba/rb_ws/src/robowflex/robowflex_dart/inc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; visual mesh filename=file:///home/serboba/rb_ws/src/robowflex/robowflex_dart/inc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
- link bellows_link: geometry collision mesh filename=file:///home/serboba/rb_ws/src/robowflex/robowflex_dart/inc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; visual mesh filename=file:///home/serboba/rb_ws/src/robowflex/robowflex_dart/inc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
- link bellows_link2: geometry collision mesh filename=file:///home/serboba/rb_ws/src/robowflex/robowflex_dart/inc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; visual mesh filename=file:///home/serboba/rb_ws/src/robowflex/robowflex_dart/inc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
- link elbow_flex_link: geometry collision mesh filename=file:///home/serboba/rb_ws/src/robowflex/robowflex_dart/inc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; visual mesh filename=file:///home/serboba/rb_ws/src/robowflex/robowflex_dart/inc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
- link estop_link: geometry collision mesh filename=file:///home/serboba/rb_ws/src/robowflex/robowflex_dart/inc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; visual mesh filename=file:///home/serboba/rb_ws/src/robowflex/robowflex_dart/inc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
- link forearm_roll_link: geometry collision mesh filename=file:///home/serboba/rb_ws/src/robowflex/robowflex_dart/inc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; visual mesh filename=file:///home/serboba/rb_ws/src/robowflex/robowflex_dart/inc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
- link gripper_link: geometry collision mesh filename=file:///home/serboba/rb_ws/src/robowflex/robowflex_dart/inc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; visual mesh filename=file:///home/serboba/rb_ws/src/robowflex/robowflex_dart/inc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
- link head_pan_link: geometry collision mesh filename=file:///home/serboba/rb_ws/src/robowflex/robowflex_dart/inc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; visual mesh filename=file:///home/serboba/rb_ws/src/robowflex/robowflex_dart/inc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
- link head_tilt_link: geometry collision mesh filename=file:///home/serboba/rb_ws/src/robowflex/robowflex_dart/inc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; visual mesh filename=file:///home/serboba/rb_ws/src/robowflex/robowflex_dart/inc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
- link l_gripper_finger_link: geometry collision mesh filename=file:///home/serboba/rb_ws/src/robowflex/robowflex_dart/inc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; visual mesh filename=file:///home/serboba/rb_ws/src/robowflex/robowflex_dart/inc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
- link l_wheel_link: geometry collision mesh filename=file:///home/serboba/rb_ws/src/robowflex/robowflex_dart/inc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; visual mesh filename=file:///home/serboba/rb_ws/src/robowflex/robowflex_dart/inc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
- link laser_link: geometry collision mesh filename=file:///home/serboba/rb_ws/src/robowflex/robowflex_dart/inc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; visual mesh filename=file:///home/serboba/rb_ws/src/robowflex/robowflex_dart/inc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
- link r_gripper_finger_link: geometry collision mesh filename=file:///home/serboba/rb_ws/src/robowflex/robowflex_dart/inc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; visual mesh filename=file:///home/serboba/rb_ws/src/robowflex/robowflex_dart/inc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
- link r_wheel_link: geometry collision mesh filename=file:///home/serboba/rb_ws/src/robowflex/robowflex_dart/inc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; visual mesh filename=file:///home/serboba/rb_ws/src/robowflex/robowflex_dart/inc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
- link shoulder_lift_link: geometry collision mesh filename=file:///home/serboba/rb_ws/src/robowflex/robowflex_dart/inc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; visual mesh filename=file:///home/serboba/rb_ws/src/robowflex/robowflex_dart/inc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
- link shoulder_pan_link: geometry collision mesh filename=file:///home/serboba/rb_ws/src/robowflex/robowflex_dart/inc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; visual mesh filename=file:///home/serboba/rb_ws/src/robowflex/robowflex_dart/inc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
- link torso_fixed_link: geometry collision mesh filename=file:///home/serboba/rb_ws/src/robowflex/robowflex_dart/inc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; visual mesh filename=file:///home/serboba/rb_ws/src/robowflex/robowflex_dart/inc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
- link torso_lift_link: geometry collision mesh filename=file:///home/serboba/rb_ws/src/robowflex/robowflex_dart/inc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; visual mesh filename=file:///home/serboba/rb_ws/src/robowflex/robowflex_dart/inc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
- link upperarm_roll_link: geometry collision mesh filename=file:///home/serboba/rb_ws/src/robowflex/robowflex_dart/inc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; visual mesh filename=file:///home/serboba/rb_ws/src/robowflex/robowflex_dart/inc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
- link wrist_flex_link: geometry collision mesh filename=file:///home/serboba/rb_ws/src/robowflex/robowflex_dart/inc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; visual mesh filename=file:///home/serboba/rb_ws/src/robowflex/robowflex_dart/inc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
- link wrist_roll_link: geometry collision mesh filename=file:///home/serboba/rb_ws/src/robowflex/robowflex_dart/inc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; visual mesh filename=file:///home/serboba/rb_ws/src/robowflex/robowflex_dart/inc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
Joints:
- joint move_x_axis_joint: limit lower=-5.0 upper=5.0 effort=10 velocity=20 -> lower=-1.1 upper=2.1 effort=10 velocity=20
- joint move_y_axis_joint: limit lower=-5.0 upper=5.0 effort=10 velocity=20 -> lower=-1.5 upper=1.2 effort=10 velocity=20

File: robowflex_dart/include/io/envs/maze1/urdf/maze1.urdf (robot description, URDF)
Before this commit: robot maze1, 8 links, 7 joints
Links:
- link link_2_joint_0: geometry collision box size=0.5 0.03 0.173; visual box size=0.5 0.03 0.173
- link table: geometry collision mesh filename=file:///home/serboba/rb_ws/src/robowflex/robowflex_dart/inc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 scale=0.50 0.50 0.50; visual mesh filename=file:///home/serboba/rb_ws/src/robowflex/robowflex_dart/inc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 scale=0.50 0.50 0.50
Joints:
- joint link_2_joint_0: origin xyz=1.25 -0.575 0.755 rpy=0 0 -1.57 -> xyz=1.25 -0.575 0.755 rpy=0 0 0

File: robowflex_dart/include/io/envs/maze3/urdf/maze3.urdf (robot description, URDF)
Before this commit: robot maze3, 9 links, 8 joints
Links:
- link table: geometry collision mesh filename=file:///home/serboba/rb_ws/src/robowflex/robowflex_dart/inc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 scale=0.750 0.750 0.750; visual mesh filename=file:///home/serboba/rb_ws/src/robowflex/robowflex_dart/inc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 scale=0.750 0.750 0.750

File: robowflex_dart/include/io/envs/room0/urdf/room0.urdf (robot description, URDF)
Before this commit: robot room0, 13 links, 12 joints
Links:
- link link_2_joint_0: geometry collision box size=0.03 0.45 0.146; visual box size=0.03 0.45 0.146
- link link_3_joint_0: geometry collision box size=1.1 0.7 0.1; visual box size=1.1 0.7 0.1
Joints:
- joint link_2_joint_0: axis 0 0 1 -> 1 0 0; origin xyz=1.30 -0.4 0.55 rpy=0 0 0 -> xyz=1.22 0.45 0.90 rpy=0 0 0
- joint link_3_joint_0: axis 1 0 0 -> 0 0 1; limit lower=0 upper=1.57 effort=0.05 velocity=1.57 -> lower=0.0 upper=1.57 effort=0.05 velocity=1.57; origin xyz=1.22 0.45 0.90 rpy=0 0 0 -> xyz=1.30 -0.4 0.55 rpy=0 0 0

File: robowflex_dart/include/io/envs/room1/urdf/room1.urdf (robot description, URDF)
Before this commit: robot room1, 13 links, 12 joints
Links:
- link link_2_joint_0: geometry collision box size=0.03 0.45 0.146; visual box size=0.03 0.45 0.146
- link link_3_joint_0: geometry collision box size=1.1 0.7 0.1; visual box size=1.1 0.7 0.1
Joints:
- joint link_2_joint_0: axis 0 0 1 -> 1 0 0; origin xyz=1.30 -0.4 0.55 rpy=0 0 0 -> xyz=1.22 0.45 0.90 rpy=0 0 0
- joint link_3_joint_0: axis 1 0 0 -> 0 0 1; limit lower=0 upper=1.57 effort=0.05 velocity=1.57 -> lower=0.0 upper=1.57 effort=0.05 velocity=1.57; origin xyz=1.22 0.45 0.90 rpy=0 0 0 -> xyz=1.30 -0.4 0.55 rpy=0 0 0
