Commit message: small bug fixes for compile

File: robowflex_dart/include/io/envs/fetch/urdf/fetch0.urdf (robot description, URDF)
Before this commit: robot fetch, 28 links, 27 joints
Links:
- link base_link: geometry collision mesh filename=/home/serboba/rb_ws/robowflex/robowflex_dart/include/io/env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; visual mesh filename=/home/serboba/rb_ws/robowflex/robowflex_dart/include/io/env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
- link bellows_link: geometry collision mesh filename=/home/serboba/rb_ws/robowflex/robowflex_dart/include/io/env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; visual mesh filename=/home/serboba/rb_ws/robowflex/robowflex_dart/include/io/env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
- link bellows_link2: geometry collision mesh filename=/home/serboba/rb_ws/robowflex/robowflex_dart/include/io/env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; visual mesh filename=/home/serboba/rb_ws/robowflex/robowflex_dart/include/io/env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
- link elbow_flex_link: geometry collision mesh filename=/home/serboba/rb_ws/robowflex/robowflex_dart/include/io/env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; visual mesh filename=/home/serboba/rb_ws/robowflex/robowflex_dart/include/io/env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
- link estop_link: geometry collision mesh filename=/home/serboba/rb_ws/robowflex/robowflex_dart/include/io/env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; visual mesh filename=/home/serboba/rb_ws/robowflex/robowflex_dart/include/io/env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
- link forearm_roll_link: geometry collision mesh filename=/home/serboba/rb_ws/robowflex/robowflex_dart/include/io/env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; visual mesh filename=/home/serboba/rb_ws/robowflex/robowflex_dart/include/io/env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
- link gripper_link: geometry collision mesh filename=/home/serboba/rb_ws/robowflex/robowflex_dart/include/io/env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; visual mesh filename=/home/serboba/rb_ws/robowflex/robowflex_dart/include/io/env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
- link head_pan_link: geometry collision mesh filename=/home/serboba/rb_ws/robowflex/robowflex_dart/include/io/env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; visual mesh filename=/home/serboba/rb_ws/robowflex/robowflex_dart/include/io/env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
- link head_tilt_link: geometry collision mesh filename=/home/serboba/rb_ws/robowflex/robowflex_dart/include/io/env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; visual mesh filename=/home/serboba/rb_ws/robowflex/robowflex_dart/include/io/env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
- link l_gripper_finger_link: geometry collision mesh filename=/home/serboba/rb_ws/robowflex/robowflex_dart/include/io/env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; visual mesh filename=/home/serboba/rb_ws/robowflex/robowflex_dart/include/io/env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
- link l_wheel_link: geometry collision mesh filename=/home/serboba/rb_ws/robowflex/robowflex_dart/include/io/env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; visual mesh filename=/home/serboba/rb_ws/robowflex/robowflex_dart/include/io/env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
- link laser_link: geometry collision mesh filename=/home/serboba/rb_ws/robowflex/robowflex_dart/include/io/env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; visual mesh filename=/home/serboba/rb_ws/robowflex/robowflex_dart/include/io/env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
- link r_gripper_finger_link: geometry collision mesh filename=/home/serboba/rb_ws/robowflex/robowflex_dart/include/io/env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; visual mesh filename=/home/serboba/rb_ws/robowflex/robowflex_dart/include/io/env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
- link r_wheel_link: geometry collision mesh filename=/home/serboba/rb_ws/robowflex/robowflex_dart/include/io/env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; visual mesh filename=/home/serboba/rb_ws/robowflex/robowflex_dart/include/io/env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
- link shoulder_lift_link: geometry collision mesh filename=/home/serboba/rb_ws/robowflex/robowflex_dart/include/io/env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; visual mesh filename=/home/serboba/rb_ws/robowflex/robowflex_dart/include/io/env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
- link shoulder_pan_link: geometry collision mesh filename=/home/serboba/rb_ws/robowflex/robowflex_dart/include/io/env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; visual mesh filename=/home/serboba/rb_ws/robowflex/robowflex_dart/include/io/env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
- link torso_fixed_link: geometry collision mesh filename=/home/serboba/rb_ws/robowflex/robowflex_dart/include/io/env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; visual mesh filename=/home/serboba/rb_ws/robowflex/robowflex_dart/include/io/env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
- link torso_lift_link: geometry collision mesh filename=/home/serboba/rb_ws/robowflex/robowflex_dart/include/io/env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; visual mesh filename=/home/serboba/rb_ws/robowflex/robowflex_dart/include/io/env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
- link upperarm_roll_link: geometry collision mesh filename=/home/serboba/rb_ws/robowflex/robowflex_dart/include/io/env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; visual mesh filename=/home/serboba/rb_ws/robowflex/robowflex_dart/include/io/env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
- link wrist_flex_link: geometry collision mesh filename=/home/serboba/rb_ws/robowflex/robowflex_dart/include/io/env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; visual mesh filename=/home/serboba/rb_ws/robowflex/robowflex_dart/include/io/env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
- link wrist_roll_link: geometry collision mesh filename=/home/serboba/rb_ws/robowflex/robowflex_dart/include/io/env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; visual mesh filename=/home/serboba/rb_ws/robowflex/robowflex_dart/include/io/env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

File: robowflex_dart/include/io/envs/fetch/urdf/fetch2.urdf (robot description, URDF)
Before this commit: robot fetch, 28 links, 27 joints
Links:
- link base_link: geometry collision mesh filename=/home/serboba/rb_ws/robowflex/robowflex_dart/include/io/env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; visual mesh filename=/home/serboba/rb_ws/robowflex/robowflex_dart/include/io/env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
- link bellows_link: geometry collision mesh filename=/home/serboba/rb_ws/robowflex/robowflex_dart/include/io/env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; visual mesh filename=/home/serboba/rb_ws/robowflex/robowflex_dart/include/io/env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
- link bellows_link2: geometry collision mesh filename=/home/serboba/rb_ws/robowflex/robowflex_dart/include/io/env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; visual mesh filename=/home/serboba/rb_ws/robowflex/robowflex_dart/include/io/env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
- link elbow_flex_link: geometry collision mesh filename=/home/serboba/rb_ws/robowflex/robowflex_dart/include/io/env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; visual mesh filename=/home/serboba/rb_ws/robowflex/robowflex_dart/include/io/env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
- link estop_link: geometry collision mesh filename=/home/serboba/rb_ws/robowflex/robowflex_dart/include/io/env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; visual mesh filename=/home/serboba/rb_ws/robowflex/robowflex_dart/include/io/env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
- link forearm_roll_link: geometry collision mesh filename=/home/serboba/rb_ws/robowflex/robowflex_dart/include/io/env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; visual mesh filename=/home/serboba/rb_ws/robowflex/robowflex_dart/include/io/env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
- link gripper_link: geometry collision mesh filename=/home/serboba/rb_ws/robowflex/robowflex_dart/include/io/env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; visual mesh filename=/home/serboba/rb_ws/robowflex/robowflex_dart/include/io/env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
- link head_pan_link: geometry collision mesh filename=/home/serboba/rb_ws/robowflex/robowflex_dart/include/io/env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; visual mesh filename=/home/serboba/rb_ws/robowflex/robowflex_dart/include/io/env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
- link head_tilt_link: geometry collision mesh filename=/home/serboba/rb_ws/robowflex/robowflex_dart/include/io/env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; visual mesh filename=/home/serboba/rb_ws/robowflex/robowflex_dart/include/io/env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
- link l_gripper_finger_link: geometry collision mesh filename=/home/serboba/rb_ws/robowflex/robowflex_dart/include/io/env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; visual mesh filename=/home/serboba/rb_ws/robowflex/robowflex_dart/include/io/env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
- link l_wheel_link: geometry collision mesh filename=/home/serboba/rb_ws/robowflex/robowflex_dart/include/io/env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; visual mesh filename=/home/serboba/rb_ws/robowflex/robowflex_dart/include/io/env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
- link laser_link: geometry collision mesh filename=/home/serboba/rb_ws/robowflex/robowflex_dart/include/io/env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; visual mesh filename=/home/serboba/rb_ws/robowflex/robowflex_dart/include/io/env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
- link r_gripper_finger_link: geometry collision mesh filename=/home/serboba/rb_ws/robowflex/robowflex_dart/include/io/env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; visual mesh filename=/home/serboba/rb_ws/robowflex/robowflex_dart/include/io/env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
- link r_wheel_link: geometry collision mesh filename=/home/serboba/rb_ws/robowflex/robowflex_dart/include/io/env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; visual mesh filename=/home/serboba/rb_ws/robowflex/robowflex_dart/include/io/env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
- link shoulder_lift_link: geometry collision mesh filename=/home/serboba/rb_ws/robowflex/robowflex_dart/include/io/env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; visual mesh filename=/home/serboba/rb_ws/robowflex/robowflex_dart/include/io/env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
- link shoulder_pan_link: geometry collision mesh filename=/home/serboba/rb_ws/robowflex/robowflex_dart/include/io/env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; visual mesh filename=/home/serboba/rb_ws/robowflex/robowflex_dart/include/io/env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
- link torso_fixed_link: geometry collision mesh filename=/home/serboba/rb_ws/robowflex/robowflex_dart/include/io/env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; visual mesh filename=/home/serboba/rb_ws/robowflex/robowflex_dart/include/io/env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
- link torso_lift_link: geometry collision mesh filename=/home/serboba/rb_ws/robowflex/robowflex_dart/include/io/env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; visual mesh filename=/home/serboba/rb_ws/robowflex/robowflex_dart/include/io/env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
- link upperarm_roll_link: geometry collision mesh filename=/home/serboba/rb_ws/robowflex/robowflex_dart/include/io/env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; visual mesh filename=/home/serboba/rb_ws/robowflex/robowflex_dart/include/io/env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
- link wrist_flex_link: geometry collision mesh filename=/home/serboba/rb_ws/robowflex/robowflex_dart/include/io/env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; visual mesh filename=/home/serboba/rb_ws/robowflex/robowflex_dart/include/io/env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
- link wrist_roll_link: geometry collision mesh filename=/home/serboba/rb_ws/robowflex/robowflex_dart/include/io/env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; visual mesh filename=/home/serboba/rb_ws/robowflex/robowflex_dart/include/io/env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

File: robowflex_dart/include/io/envs/fetch/urdf/fetch3.urdf (robot description, URDF)
Before this commit: robot fetch, 28 links, 27 joints
Links:
- link base_link: geometry collision mesh filename=/home/serboba/rb_ws/robowflex/robowflex_dart/include/io/env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; visual mesh filename=/home/serboba/rb_ws/robowflex/robowflex_dart/include/io/env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
- link bellows_link: geometry collision mesh filename=/home/serboba/rb_ws/robowflex/robowflex_dart/include/io/env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; visual mesh filename=/home/serboba/rb_ws/robowflex/robowflex_dart/include/io/env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
- link bellows_link2: geometry collision mesh filename=/home/serboba/rb_ws/robowflex/robowflex_dart/include/io/env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; visual mesh filename=/home/serboba/rb_ws/robowflex/robowflex_dart/include/io/env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
- link elbow_flex_link: geometry collision mesh filename=/home/serboba/rb_ws/robowflex/robowflex_dart/include/io/env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; visual mesh filename=/home/serboba/rb_ws/robowflex/robowflex_dart/include/io/env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
- link estop_link: geometry collision mesh filename=/home/serboba/rb_ws/robowflex/robowflex_dart/include/io/env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; visual mesh filename=/home/serboba/rb_ws/robowflex/robowflex_dart/include/io/env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
- link forearm_roll_link: geometry collision mesh filename=/home/serboba/rb_ws/robowflex/robowflex_dart/include/io/env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; visual mesh filename=/home/serboba/rb_ws/robowflex/robowflex_dart/include/io/env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
- link gripper_link: geometry collision mesh filename=/home/serboba/rb_ws/robowflex/robowflex_dart/include/io/env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; visual mesh filename=/home/serboba/rb_ws/robowflex/robowflex_dart/include/io/env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
- link head_pan_link: geometry collision mesh filename=/home/serboba/rb_ws/robowflex/robowflex_dart/include/io/env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; visual mesh filename=/home/serboba/rb_ws/robowflex/robowflex_dart/include/io/env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
- link head_tilt_link: geometry collision mesh filename=/home/serboba/rb_ws/robowflex/robowflex_dart/include/io/env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; visual mesh filename=/home/serboba/rb_ws/robowflex/robowflex_dart/include/io/env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
- link l_gripper_finger_link: geometry collision mesh filename=/home/serboba/rb_ws/robowflex/robowflex_dart/include/io/env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; visual mesh filename=/home/serboba/rb_ws/robowflex/robowflex_dart/include/io/env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
- link l_wheel_link: geometry collision mesh filename=/home/serboba/rb_ws/robowflex/robowflex_dart/include/io/env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; visual mesh filename=/home/serboba/rb_ws/robowflex/robowflex_dart/include/io/env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
- link laser_link: geometry collision mesh filename=/home/serboba/rb_ws/robowflex/robowflex_dart/include/io/env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; visual mesh filename=/home/serboba/rb_ws/robowflex/robowflex_dart/include/io/env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
- link r_gripper_finger_link: geometry collision mesh filename=/home/serboba/rb_ws/robowflex/robowflex_dart/include/io/env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; visual mesh filename=/home/serboba/rb_ws/robowflex/robowflex_dart/include/io/env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
- link r_wheel_link: geometry collision mesh filename=/home/serboba/rb_ws/robowflex/robowflex_dart/include/io/env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; visual mesh filename=/home/serboba/rb_ws/robowflex/robowflex_dart/include/io/env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
- link shoulder_lift_link: geometry collision mesh filename=/home/serboba/rb_ws/robowflex/robowflex_dart/include/io/env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; visual mesh filename=/home/serboba/rb_ws/robowflex/robowflex_dart/include/io/env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
- link shoulder_pan_link: geometry collision mesh filename=/home/serboba/rb_ws/robowflex/robowflex_dart/include/io/env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; visual mesh filename=/home/serboba/rb_ws/robowflex/robowflex_dart/include/io/env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
- link torso_fixed_link: geometry collision mesh filename=/home/serboba/rb_ws/robowflex/robowflex_dart/include/io/env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; visual mesh filename=/home/serboba/rb_ws/robowflex/robowflex_dart/include/io/env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
- link torso_lift_link: geometry collision mesh filename=/home/serboba/rb_ws/robowflex/robowflex_dart/include/io/env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; visual mesh filename=/home/serboba/rb_ws/robowflex/robowflex_dart/include/io/env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
- link upperarm_roll_link: geometry collision mesh filename=/home/serboba/rb_ws/robowflex/robowflex_dart/include/io/env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; visual mesh filename=/home/serboba/rb_ws/robowflex/robowflex_dart/include/io/env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
- link wrist_flex_link: geometry collision mesh filename=/home/serboba/rb_ws/robowflex/robowflex_dart/include/io/env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; visual mesh filename=/home/serboba/rb_ws/robowflex/robowflex_dart/include/io/env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
- link wrist_roll_link: geometry collision mesh filename=/home/serboba/rb_ws/robowflex/robowflex_dart/include/io/env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; visual mesh filename=/home/serboba/rb_ws/robowflex/robowflex_dart/include/io/env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

File: robowflex_dart/include/io/envs/fetch/urdf/fetch4.urdf (robot description, URDF)
Before this commit: robot fetch, 29 links, 28 joints
Links:
- link base_link: geometry collision mesh filename=/home/serboba/rb_ws/robowflex/robowflex_dart/include/io/env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; visual mesh filename=/home/serboba/rb_ws/robowflex/robowflex_dart/include/io/env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
- link bellows_link: geometry collision mesh filename=/home/serboba/rb_ws/robowflex/robowflex_dart/include/io/env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; visual mesh filename=/home/serboba/rb_ws/robowflex/robowflex_dart/include/io/env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
- link bellows_link2: geometry collision mesh filename=/home/serboba/rb_ws/robowflex/robowflex_dart/include/io/env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; visual mesh filename=/home/serboba/rb_ws/robowflex/robowflex_dart/include/io/env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
- link elbow_flex_link: geometry collision mesh filename=/home/serboba/rb_ws/robowflex/robowflex_dart/include/io/env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; visual mesh filename=/home/serboba/rb_ws/robowflex/robowflex_dart/include/io/env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
- link estop_link: geometry collision mesh filename=/home/serboba/rb_ws/robowflex/robowflex_dart/include/io/env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; visual mesh filename=/home/serboba/rb_ws/robowflex/robowflex_dart/include/io/env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
- link forearm_roll_link: geometry collision mesh filename=/home/serboba/rb_ws/robowflex/robowflex_dart/include/io/env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; visual mesh filename=/home/serboba/rb_ws/robowflex/robowflex_dart/include/io/env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
- link gripper_link: geometry collision mesh filename=/home/serboba/rb_ws/robowflex/robowflex_dart/include/io/env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; visual mesh filename=/home/serboba/rb_ws/robowflex/robowflex_dart/include/io/env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
- link head_pan_link: geometry collision mesh filename=/home/serboba/rb_ws/robowflex/robowflex_dart/include/io/env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; visual mesh filename=/home/serboba/rb_ws/robowflex/robowflex_dart/include/io/env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
- link head_tilt_link: geometry collision mesh filename=/home/serboba/rb_ws/robowflex/robowflex_dart/include/io/env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; visual mesh filename=/home/serboba/rb_ws/robowflex/robowflex_dart/include/io/env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
- link l_gripper_finger_link: geometry collision mesh filename=/home/serboba/rb_ws/robowflex/robowflex_dart/include/io/env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; visual mesh filename=/home/serboba/rb_ws/robowflex/robowflex_dart/include/io/env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
- link l_wheel_link: geometry collision mesh filename=/home/serboba/rb_ws/robowflex/robowflex_dart/include/io/env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; visual mesh filename=/home/serboba/rb_ws/robowflex/robowflex_dart/include/io/env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
- link laser_link: geometry collision mesh filename=/home/serboba/rb_ws/robowflex/robowflex_dart/include/io/env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; visual mesh filename=/home/serboba/rb_ws/robowflex/robowflex_dart/include/io/env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
- link r_gripper_finger_link: geometry collision mesh filename=/home/serboba/rb_ws/robowflex/robowflex_dart/include/io/env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; visual mesh filename=/home/serboba/rb_ws/robowflex/robowflex_dart/include/io/env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
- link r_wheel_link: geometry collision mesh filename=/home/serboba/rb_ws/robowflex/robowflex_dart/include/io/env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; visual mesh filename=/home/serboba/rb_ws/robowflex/robowflex_dart/include/io/env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
- link shoulder_lift_link: geometry collision mesh filename=/home/serboba/rb_ws/robowflex/robowflex_dart/include/io/env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; visual mesh filename=/home/serboba/rb_ws/robowflex/robowflex_dart/include/io/env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
- link shoulder_pan_link: geometry collision mesh filename=/home/serboba/rb_ws/robowflex/robowflex_dart/include/io/env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; visual mesh filename=/home/serboba/rb_ws/robowflex/robowflex_dart/include/io/env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
- link torso_fixed_link: geometry collision mesh filename=/home/serboba/rb_ws/robowflex/robowflex_dart/include/io/env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; visual mesh filename=/home/serboba/rb_ws/robowflex/robowflex_dart/include/io/env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
- link torso_lift_link: geometry collision mesh filename=/home/serboba/rb_ws/robowflex/robowflex_dart/include/io/env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; visual mesh filename=/home/serboba/rb_ws/robowflex/robowflex_dart/include/io/env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
- link upperarm_roll_link: geometry collision mesh filename=/home/serboba/rb_ws/robowflex/robowflex_dart/include/io/env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; visual mesh filename=/home/serboba/rb_ws/robowflex/robowflex_dart/include/io/env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
- link wrist_flex_link: geometry collision mesh filename=/home/serboba/rb_ws/robowflex/robowflex_dart/include/io/env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; visual mesh filename=/home/serboba/rb_ws/robowflex/robowflex_dart/include/io/env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
- link wrist_roll_link: geometry collision mesh filename=/home/serboba/rb_ws/robowflex/robowflex_dart/include/io/env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; visual mesh filename=/home/serboba/rb_ws/robowflex/robowflex_dart/include/io/env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

File: robowflex_dart/include/io/envs/fetch/urdf/fetch5.urdf (robot description, URDF)
Before this commit: robot fetch, 29 links, 28 joints
Links:
- link base_link: geometry collision mesh filename=/home/serboba/rb_ws/robowflex/robowflex_dart/include/io/env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; visual mesh filename=/home/serboba/rb_ws/robowflex/robowflex_dart/include/io/env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
- link bellows_link: geometry collision mesh filename=/home/serboba/rb_ws/robowflex/robowflex_dart/include/io/env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; visual mesh filename=/home/serboba/rb_ws/robowflex/robowflex_dart/include/io/env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
- link bellows_link2: geometry collision mesh filename=/home/serboba/rb_ws/robowflex/robowflex_dart/include/io/env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; visual mesh filename=/home/serboba/rb_ws/robowflex/robowflex_dart/include/io/env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
- link elbow_flex_link: geometry collision mesh filename=/home/serboba/rb_ws/robowflex/robowflex_dart/include/io/env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; visual mesh filename=/home/serboba/rb_ws/robowflex/robowflex_dart/include/io/env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
- link estop_link: geometry collision mesh filename=/home/serboba/rb_ws/robowflex/robowflex_dart/include/io/env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; visual mesh filename=/home/serboba/rb_ws/robowflex/robowflex_dart/include/io/env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
- link forearm_roll_link: geometry collision mesh filename=/home/serboba/rb_ws/robowflex/robowflex_dart/include/io/env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; visual mesh filename=/home/serboba/rb_ws/robowflex/robowflex_dart/include/io/env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
- link gripper_link: geometry collision mesh filename=/home/serboba/rb_ws/robowflex/robowflex_dart/include/io/env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; visual mesh filename=/home/serboba/rb_ws/robowflex/robowflex_dart/include/io/env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
- link head_pan_link: geometry collision mesh filename=/home/serboba/rb_ws/robowflex/robowflex_dart/include/io/env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; visual mesh filename=/home/serboba/rb_ws/robowflex/robowflex_dart/include/io/env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
- link head_tilt_link: geometry collision mesh filename=/home/serboba/rb_ws/robowflex/robowflex_dart/include/io/env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; visual mesh filename=/home/serboba/rb_ws/robowflex/robowflex_dart/include/io/env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
- link l_gripper_finger_link: geometry collision mesh filename=/home/serboba/rb_ws/robowflex/robowflex_dart/include/io/env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; visual mesh filename=/home/serboba/rb_ws/robowflex/robowflex_dart/include/io/env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
- link l_wheel_link: geometry collision mesh filename=/home/serboba/rb_ws/robowflex/robowflex_dart/include/io/env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; visual mesh filename=/home/serboba/rb_ws/robowflex/robowflex_dart/include/io/env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
- link laser_link: geometry collision mesh filename=/home/serboba/rb_ws/robowflex/robowflex_dart/include/io/env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; visual mesh filename=/home/serboba/rb_ws/robowflex/robowflex_dart/include/io/env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
- link r_gripper_finger_link: geometry collision mesh filename=/home/serboba/rb_ws/robowflex/robowflex_dart/include/io/env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; visual mesh filename=/home/serboba/rb_ws/robowflex/robowflex_dart/include/io/env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
- link r_wheel_link: geometry collision mesh filename=/home/serboba/rb_ws/robowflex/robowflex_dart/include/io/env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; visual mesh filename=/home/serboba/rb_ws/robowflex/robowflex_dart/include/io/env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
- link shoulder_lift_link: geometry collision mesh filename=/home/serboba/rb_ws/robowflex/robowflex_dart/include/io/env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; visual mesh filename=/home/serboba/rb_ws/robowflex/robowflex_dart/include/io/env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
- link shoulder_pan_link: geometry collision mesh filename=/home/serboba/rb_ws/robowflex/robowflex_dart/include/io/env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; visual mesh filename=/home/serboba/rb_ws/robowflex/robowflex_dart/include/io/env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
- link torso_fixed_link: geometry collision mesh filename=/home/serboba/rb_ws/robowflex/robowflex_dart/include/io/env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; visual mesh filename=/home/serboba/rb_ws/robowflex/robowflex_dart/include/io/env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
- link torso_lift_link: geometry collision mesh filename=/home/serboba/rb_ws/robowflex/robowflex_dart/include/io/env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; visual mesh filename=/home/serboba/rb_ws/robowflex/robowflex_dart/include/io/env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
- link upperarm_roll_link: geometry collision mesh filename=/home/serboba/rb_ws/robowflex/robowflex_dart/include/io/env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; visual mesh filename=/home/serboba/rb_ws/robowflex/robowflex_dart/include/io/env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
- link wrist_flex_link: geometry collision mesh filename=/home/serboba/rb_ws/robowflex/robowflex_dart/include/io/env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; visual mesh filename=/home/serboba/rb_ws/robowflex/robowflex_dart/include/io/env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
- link wrist_roll_link: geometry collision mesh filename=/home/serboba/rb_ws/robowflex/robowflex_dart/include/io/env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; visual mesh filename=/home/serboba/rb_ws/robowflex/robowflex_dart/include/io/env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
