Commit message: small bug fixes for compile

File: robowflex_dart/include/io/envs/fetch/urdf/fetch6.urdf (robot description, URDF)
Before this commit: robot fetch, 29 links, 28 joints
Links:
- link base_link: geometry collision mesh filename=/home/serboba/rb_ws/robowflex/robowflex_dart/include/io/env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; visual mesh filename=/home/serboba/rb_ws/robowflex/robowflex_dart/include/io/env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
- link bellows_link: geometry collision mesh filename=/home/serboba/rb_ws/robowflex/robowflex_dart/include/io/env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; visual mesh filename=/home/serboba/rb_ws/robowflex/robowflex_dart/include/io/env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
- link bellows_link2: geometry collision mesh filename=/home/serboba/rb_ws/robowflex/robowflex_dart/include/io/env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; visual mesh filename=/home/serboba/rb_ws/robowflex/robowflex_dart/include/io/env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
- link elbow_flex_link: geometry collision mesh filename=/home/serboba/rb_ws/robowflex/robowflex_dart/include/io/env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; visual mesh filename=/home/serboba/rb_ws/robowflex/robowflex_dart/include/io/env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
- link estop_link: geometry collision mesh filename=/home/serboba/rb_ws/robowflex/robowflex_dart/include/io/env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; visual mesh filename=/home/serboba/rb_ws/robowflex/robowflex_dart/include/io/env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
- link forearm_roll_link: geometry collision mesh filename=/home/serboba/rb_ws/robowflex/robowflex_dart/include/io/env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; visual mesh filename=/home/serboba/rb_ws/robowflex/robowflex_dart/include/io/env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
- link gripper_link: geometry collision mesh filename=/home/serboba/rb_ws/robowflex/robowflex_dart/include/io/env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; visual mesh filename=/home/serboba/rb_ws/robowflex/robowflex_dart/include/io/env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
- link head_pan_link: geometry collision mesh filename=/home/serboba/rb_ws/robowflex/robowflex_dart/include/io/env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; visual mesh filename=/home/serboba/rb_ws/robowflex/robowflex_dart/include/io/env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
- link head_tilt_link: geometry collision mesh filename=/home/serboba/rb_ws/robowflex/robowflex_dart/include/io/env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; visual mesh filename=/home/serboba/rb_ws/robowflex/robowflex_dart/include/io/env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
- link l_gripper_finger_link: geometry collision mesh filename=/home/serboba/rb_ws/robowflex/robowflex_dart/include/io/env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; visual mesh filename=/home/serboba/rb_ws/robowflex/robowflex_dart/include/io/env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
- link l_wheel_link: geometry collision mesh filename=/home/serboba/rb_ws/robowflex/robowflex_dart/include/io/env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; visual mesh filename=/home/serboba/rb_ws/robowflex/robowflex_dart/include/io/env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
- link laser_link: geometry collision mesh filename=/home/serboba/rb_ws/robowflex/robowflex_dart/include/io/env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; visual mesh filename=/home/serboba/rb_ws/robowflex/robowflex_dart/include/io/env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
- link r_gripper_finger_link: geometry collision mesh filename=/home/serboba/rb_ws/robowflex/robowflex_dart/include/io/env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; visual mesh filename=/home/serboba/rb_ws/robowflex/robowflex_dart/include/io/env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
- link r_wheel_link: geometry collision mesh filename=/home/serboba/rb_ws/robowflex/robowflex_dart/include/io/env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; visual mesh filename=/home/serboba/rb_ws/robowflex/robowflex_dart/include/io/env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
- link shoulder_lift_link: geometry collision mesh filename=/home/serboba/rb_ws/robowflex/robowflex_dart/include/io/env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; visual mesh filename=/home/serboba/rb_ws/robowflex/robowflex_dart/include/io/env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
- link shoulder_pan_link: geometry collision mesh filename=/home/serboba/rb_ws/robowflex/robowflex_dart/include/io/env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; visual mesh filename=/home/serboba/rb_ws/robowflex/robowflex_dart/include/io/env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
- link torso_fixed_link: geometry collision mesh filename=/home/serboba/rb_ws/robowflex/robowflex_dart/include/io/env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; visual mesh filename=/home/serboba/rb_ws/robowflex/robowflex_dart/include/io/env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
- link torso_lift_link: geometry collision mesh filename=/home/serboba/rb_ws/robowflex/robowflex_dart/include/io/env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; visual mesh filename=/home/serboba/rb_ws/robowflex/robowflex_dart/include/io/env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
- link upperarm_roll_link: geometry collision mesh filename=/home/serboba/rb_ws/robowflex/robowflex_dart/include/io/env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; visual mesh filename=/home/serboba/rb_ws/robowflex/robowflex_dart/include/io/env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
- link wrist_flex_link: geometry collision mesh filename=/home/serboba/rb_ws/robowflex/robowflex_dart/include/io/env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; visual mesh filename=/home/serboba/rb_ws/robowflex/robowflex_dart/include/io/env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
- link wrist_roll_link: geometry collision mesh filename=/home/serboba/rb_ws/robowflex/robowflex_dart/include/io/env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; visual mesh filename=/home/serboba/rb_ws/robowflex/robowflex_dart/include/io/env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

File: robowflex_dart/include/io/envs/maze1/urdf/maze1.urdf (robot description, URDF)
Before this commit: robot maze1, 8 links, 7 joints
Links:
- link table: geometry collision mesh filename=/home/serboba/rb_ws/robowflex/robowflex_dart/include/io/env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 scale=0.50 0.50 0.50; visual mesh filename=/home/serboba/rb_ws/robowflex/robowflex_dart/include/io/env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 scale=0.50 0.50 0.50

File: robowflex_dart/include/io/envs/maze2/urdf/maze2.urdf (robot description, URDF)
Before this commit: robot maze2, 9 links, 8 joints
Links:
- link table: geometry collision mesh filename=/home/serboba/rb_ws/robowflex/robowflex_dart/include/io/env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 scale=0.750 0.750 0.750; visual mesh filename=/home/serboba/rb_ws/robowflex/robowflex_dart/include/io/env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 scale=0.750 0.750 0.750

File: robowflex_dart/include/io/envs/maze3/urdf/maze3.urdf (robot description, URDF)
Before this commit: robot maze3, 9 links, 8 joints
Links:
- link table: geometry collision mesh filename=/home/serboba/rb_ws/robowflex/robowflex_dart/include/io/env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 scale=0.750 0.750 0.750; visual mesh filename=/home/serboba/rb_ws/robowflex/robowflex_dart/include/io/env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 scale=0.750 0.750 0.750

File: robowflex_dart/include/io/envs/maze_vertical/urdf/maze_vertical.urdf (robot description, URDF)
Before this commit: robot maze_vertical, 9 links, 8 joints
Links:
- link table: geometry collision mesh filename=/home/serboba/rb_ws/robowflex/robowflex_dart/include/io/env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 scale=0.50 0.50 0.50; visual mesh filename=/home/serboba/rb_ws/robowflex/robowflex_dart/include/io/env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 scale=0.50 0.50 0.50

File: robowflex_dart/include/io/envs/room/urdf/room.urdf (robot description, URDF)
Before this commit: robot room, 13 links, 12 joints
Links:
- link desk: geometry collision mesh filename=/home/serboba/rb_ws/robowflex/robowflex_dart/include/io/env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 scale=0.01 0.01 0.020; visual mesh filename=/home/serboba/rb_ws/robowflex/robowflex_dart/include/io/env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 scale=0.01 0.01 0.020
- link room: geometry collision mesh filename=/home/serboba/rb_ws/robowflex/robowflex_dart/include/io/env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 scale=0.4 0.4 0.3; visual mesh filename=/home/serboba/rb_ws/robowflex/robowflex_dart/include/io/env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 scale=0.4 0.4 0.3
- link shelf: geometry collision mesh filename=/home/serboba/rb_ws/robowflex/robowflex_dart/include/io/env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 scale=0.042 0.05 0.04; visual mesh filename=/home/serboba/rb_ws/robowflex/robowflex_dart/include/io/env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 scale=0.042 0.05 0.04
- link sofa: geometry collision mesh filename=/home/serboba/rb_ws/robowflex/robowflex_dart/include/io/env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 scale=0.7 0.7 1; visual mesh filename=/home/serboba/rb_ws/robowflex/robowflex_dart/include/io/env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 scale=0.7 0.7 1

File: robowflex_dart/include/io/envs/room0/urdf/room0.urdf (robot description, URDF)
Before this commit: robot room0, 13 links, 12 joints
Links:
- link desk: geometry collision mesh filename=/home/serboba/rb_ws/robowflex/robowflex_dart/include/io/env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 scale=0.01 0.01 0.020; visual mesh filename=/home/serboba/rb_ws/robowflex/robowflex_dart/include/io/env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 scale=0.01 0.01 0.020
- link room: geometry collision mesh filename=/home/serboba/rb_ws/robowflex/robowflex_dart/include/io/env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 scale=0.4 0.4 0.3; visual mesh filename=/home/serboba/rb_ws/robowflex/robowflex_dart/include/io/env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 scale=0.4 0.4 0.3
- link shelf: geometry collision mesh filename=/home/serboba/rb_ws/robowflex/robowflex_dart/include/io/env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 scale=0.042 0.05 0.04; visual mesh filename=/home/serboba/rb_ws/robowflex/robowflex_dart/include/io/env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 scale=0.042 0.05 0.04
- link sofa: geometry collision mesh filename=/home/serboba/rb_ws/robowflex/robowflex_dart/include/io/env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 scale=0.7 0.7 1; visual mesh filename=/home/serboba/rb_ws/robowflex/robowflex_dart/include/io/env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 scale=0.7 0.7 1

File: robowflex_dart/include/io/envs/room0/urdf/room01.urdf (robot description, URDF)
Before this commit: robot room0, 13 links, 12 joints
Links:
- link desk: geometry collision mesh filename=/home/serboba/rb_ws/robowflex/robowflex_dart/include/io/env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 scale=0.01 0.01 0.020; visual mesh filename=/home/serboba/rb_ws/robowflex/robowflex_dart/include/io/env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 scale=0.01 0.01 0.020
- link room: geometry collision mesh filename=/home/serboba/rb_ws/robowflex/robowflex_dart/include/io/env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 scale=0.4 0.4 0.3; visual mesh filename=/home/serboba/rb_ws/robowflex/robowflex_dart/include/io/env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 scale=0.4 0.4 0.3
- link shelf: geometry collision mesh filename=/home/serboba/rb_ws/robowflex/robowflex_dart/include/io/env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 scale=0.042 0.05 0.04; visual mesh filename=/home/serboba/rb_ws/robowflex/robowflex_dart/include/io/env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 scale=0.042 0.05 0.04
- link sofa: geometry collision mesh filename=/home/serboba/rb_ws/robowflex/robowflex_dart/include/io/env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 scale=0.7 0.7 1; visual mesh filename=/home/serboba/rb_ws/robowflex/robowflex_dart/include/io/env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 scale=0.7 0.7 1

File: robowflex_dart/include/io/envs/room0/urdf/roomcorect.urdf (robot description, URDF)
Before this commit: robot room0, 13 links, 12 joints
Links:
- link desk: geometry collision mesh filename=/home/serboba/rb_ws/robowflex/robowflex_dart/include/io/env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 scale=0.01 0.01 0.020; visual mesh filename=/home/serboba/rb_ws/robowflex/robowflex_dart/include/io/env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 scale=0.01 0.01 0.020
- link room: geometry collision mesh filename=/home/serboba/rb_ws/robowflex/robowflex_dart/include/io/env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 scale=0.4 0.4 0.3; visual mesh filename=/home/serboba/rb_ws/robowflex/robowflex_dart/include/io/env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 scale=0.4 0.4 0.3
- link shelf: geometry collision mesh filename=/home/serboba/rb_ws/robowflex/robowflex_dart/include/io/env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 scale=0.042 0.05 0.04; visual mesh filename=/home/serboba/rb_ws/robowflex/robowflex_dart/include/io/env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 scale=0.042 0.05 0.04
- link sofa: geometry collision mesh filename=/home/serboba/rb_ws/robowflex/robowflex_dart/include/io/env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 scale=0.7 0.7 1; visual mesh filename=/home/serboba/rb_ws/robowflex/robowflex_dart/include/io/env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 scale=0.7 0.7 1

File: robowflex_dart/include/io/envs/room1/urdf/room1.urdf (robot description, URDF)
Before this commit: robot room1, 13 links, 12 joints
Links:
- link desk: geometry collision mesh filename=/home/serboba/rb_ws/robowflex/robowflex_dart/include/io/env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 scale=0.01 0.01 0.020; visual mesh filename=/home/serboba/rb_ws/robowflex/robowflex_dart/include/io/env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 scale=0.01 0.01 0.020
- link room: geometry collision mesh filename=/home/serboba/rb_ws/robowflex/robowflex_dart/include/io/env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 scale=0.4 0.4 0.3; visual mesh filename=/home/serboba/rb_ws/robowflex/robowflex_dart/include/io/env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 scale=0.4 0.4 0.3
- link shelf: geometry collision mesh filename=/home/serboba/rb_ws/robowflex/robowflex_dart/include/io/env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 scale=0.042 0.05 0.04; visual mesh filename=/home/serboba/rb_ws/robowflex/robowflex_dart/include/io/env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 scale=0.042 0.05 0.04
- link sofa: geometry collision mesh filename=/home/serboba/rb_ws/robowflex/robowflex_dart/include/io/env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 scale=0.9 0.7 1; visual mesh filename=/home/serboba/rb_ws/robowflex/robowflex_dart/include/io/env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 scale=0.9 0.7 1

File: robowflex_dart/include/io/envs/room2/urdf/room2.urdf (robot description, URDF)
Before this commit: robot room2, 7 links, 6 joints
Links:
- link room: geometry collision mesh filename=/home/serboba/rb_ws/robowflex/robowflex_dart/include/io/env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 scale=0.4 0.4 0.3; visual mesh filename=/home/serboba/rb_ws/robowflex/robowflex_dart/include/io/env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 scale=0.4 0.4 0.3

File: robowflex_dart/include/io/envs/room3/urdf/room3.urdf (robot description, URDF)
Before this commit: robot room2, 7 links, 6 joints
Links:
- link room: geometry collision mesh filename=/home/serboba/rb_ws/robowflex/robowflex_dart/include/io/env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 scale=0.4 0.4 0.3; visual mesh filename=/home/serboba/rb_ws/robowflex/robowflex_dart/include/io/env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 scale=0.4 0.4 0.3
